Commit message: changed urdf files

File: youbot_common/youbot_description/robots/youbot-sensors.urdf.xacro (robot description, xacro)
@@ -7,17 +7,17 @@
   <!-- The following included files set up definitions of parts of the robot body -->
   <!-- misc common stuff? -->
-  <include filename="$(find youbot_description)/urdf/common.xacro" />
+  <xacro:include filename="$(find youbot_description)/urdf/common.xacro" />
   <!-- youbot base -->
-  <include filename="$(find youbot_description)/urdf/youbot_base/base.urdf.xacro" />
+  <xacro:include filename="$(find youbot_description)/urdf/youbot_base/base.urdf.xacro" />
   <!-- youbot plate -->
-  <include filename="$(find youbot_description)/urdf/youbot_plate/plate.urdf.xacro" />
+  <xacro:include filename="$(find youbot_description)/urdf/youbot_plate/plate.urdf.xacro" />
   <!-- youbot arm -->
-  <include filename="$(find youbot_description)/urdf/youbot_arm/arm.urdf.xacro"/>
+  <xacro:include filename="$(find youbot_description)/urdf/youbot_arm/arm.urdf.xacro"/>
   <!-- youbot gripper -->
-  <include filename="$(find youbot_description)/urdf/youbot_gripper/gripper.urdf.xacro" />
+  <xacro:include filename="$(find youbot_description)/urdf/youbot_gripper/gripper.urdf.xacro" />
   <!-- generic simulator_gazebo plugins for starting mechanism control, ros time, ros battery -->
-  <include filename="$(find youbot_description)/gazebo/gazebo.urdf.xacro" />
+  <xacro:include filename="$(find youbot_description)/gazebo/gazebo.urdf.xacro" />
   <!-- materials for visualization -->
-  <include filename="$(find youbot_description)/urdf/materials.urdf.xacro" />
+  <xacro:include filename="$(find youbot_description)/urdf/materials.urdf.xacro" />
   <!-- Now we can start using the macros included above to define the actual youbot -->
   <!-- The first use of a macro.  This one was defined in base.urdf.xacro above.
@@ -40,10 +40,10 @@
   </xacro:youbot_gripper>
   <!-- BRSU SPECIFIC STUFF -->
-  <include filename="$(find youbot_description)/urdf/updated_materials.urdf.xacro" />
-  <include filename="$(find youbot_description)/urdf/misc/sensor_angle.urdf.xacro" />
-  <include filename="$(find youbot_description)/urdf/misc/cam3d_tower.urdf.xacro" />
-  <include filename="$(find youbot_description)/urdf/sensors/kinect_camera.urdf.xacro" />
-  <include filename="$(find youbot_description)/urdf/sensors/microsoft_lifecam.urdf.xacro" />
-  <include filename="$(find youbot_description)/urdf/sensors/asus_xtion_camera.urdf.xacro" />
+  <xacro:include filename="$(find youbot_description)/urdf/updated_materials.urdf.xacro" />
+  <xacro:include filename="$(find youbot_description)/urdf/misc/sensor_angle.urdf.xacro" />
+  <xacro:include filename="$(find youbot_description)/urdf/misc/cam3d_tower.urdf.xacro" />
+  <xacro:include filename="$(find youbot_description)/urdf/sensors/kinect_camera.urdf.xacro" />
+  <xacro:include filename="$(find youbot_description)/urdf/sensors/microsoft_lifecam.urdf.xacro" />
+  <xacro:include filename="$(find youbot_description)/urdf/sensors/asus_xtion_camera.urdf.xacro" />
   <!-- base laser rear -->
   <xacro:hokuyo_urg04_laser name="base_laser_rear" parent="base" ros_topic="scan_rear" update_rate="10" min_angle="-1.57" max_angle="1.57">

File: youbot_common/youbot_description/robots/youbot.urdf.xacro (robot description, xacro)
@@ -3,21 +3,21 @@
        xmlns:controller="http://playerstage.sourceforge.net/gazebo/xmlschema/#controller"
        xmlns:interface="http://playerstage.sourceforge.net/gazebo/xmlschema/#interface"
-       xmlns:xacro="http://playerstage.sourceforge.net/gazebo/xmlschema/#interface"
-       name="youbot" >
+       xmlns:xacro="http://ros.org/wiki/xacro"
+       name="youbot">
   <!-- The following included files set up definitions of parts of the robot body -->
   <!-- misc common stuff? -->
-  <include filename="$(find youbot_description)/urdf/common.xacro" />
+  <xacro:include filename="$(find youbot_description)/urdf/common.xacro" />
   <!-- youbot base -->
-  <include filename="$(find youbot_description)/urdf/youbot_base/base.urdf.xacro" />
+  <xacro:include filename="$(find youbot_description)/urdf/youbot_base/base.urdf.xacro" />
   <!-- youbot plate -->
-  <include filename="$(find youbot_description)/urdf/youbot_plate/plate.urdf.xacro" />
+  <xacro:include filename="$(find youbot_description)/urdf/youbot_plate/plate.urdf.xacro" />
   <!-- youbot arm -->
-  <include filename="$(find youbot_description)/urdf/youbot_arm/arm.urdf.xacro"/>
+  <xacro:include filename="$(find youbot_description)/urdf/youbot_arm/arm.urdf.xacro"/>
   <!-- youbot gripper -->
-  <include filename="$(find youbot_description)/urdf/youbot_gripper/gripper.urdf.xacro" />
+  <xacro:include filename="$(find youbot_description)/urdf/youbot_gripper/gripper.urdf.xacro" />
   <!-- generic simulator_gazebo plugins for starting mechanism control, ros time, ros battery -->
-  <include filename="$(find youbot_description)/gazebo/gazebo.urdf.xacro" />
+  <xacro:include filename="$(find youbot_description)/gazebo/gazebo.urdf.xacro" />
   <!-- materials for visualization -->
-  <include filename="$(find youbot_description)/urdf/materials.urdf.xacro" />
+  <xacro:include filename="$(find youbot_description)/urdf/materials.urdf.xacro" />
   <!-- Now we can start using the macros included above to define the actual youbot -->
   <!-- The first use of a macro.  This one was defined in base.urdf.xacro above.

File: youbot_common/youbot_description/urdf/common.xacro (robot description, xacro)
@@ -1,9 +1,8 @@
 <?xml version="1.0"?>
-<robot>
-	<property name="M_PI" value="3.1415926535897931" />
-	<!-- Casters -->
-	<property name="cal_caster_fl" value="0.0" />
-	<property name="cal_caster_fr" value="0.0" />
-	<property name="cal_caster_bl" value="0.0" />
-	<property name="cal_caster_br" value="0.0" />
+<robot xmlns:xacro="http://ros.org/wiki/xacro" name="generic">
+	<xacro:property name="M_PI" value="3.1415926535897931"/>
+	<xacro:property name="cal_caster_fl" value="0.0"/>
+	<xacro:property name="cal_caster_fr" value="0.0"/>
+	<xacro:property name="cal_caster_bl" value="0.0"/>
+	<xacro:property name="cal_caster_br" value="0.0"/>
 </robot>

File: youbot_common/youbot_description/urdf/sensors/asus_xtion_camera.urdf.xacro (robot description, xacro)
@@ -1,7 +1,7 @@
 <?xml version="1.0"?>
 <root xmlns:xacro="http://playerstage.sourceforge.net/gazebo/xmlschema/#interface">
-  <include filename="$(find youbot_description)/urdf/sensors/asus_xtion_camera.gazebo.xacro" />
-  <property name="eye_x_offset" value="0.03" />
-  <property name="eye_y_offset" value="0.035" />
+  <xacro:include filename="$(find youbot_description)/urdf/sensors/asus_xtion_camera.gazebo.xacro" />
+  <xacro:property name="eye_x_offset" value="0.03" />
+  <xacro:property name="eye_y_offset" value="0.035" />
   <xacro:macro name="asus_xtion_eye" params="suffix parent *origin">
 	<link name="${parent}_${suffix}_frame">
@@ -15,5 +15,5 @@
 	  <parent link="${parent}_camera"/>
 	  <child link="${parent}_${suffix}_frame"/>
-	  <insert_block name="origin"/>
+	  <xacro:insert_block name="origin"/>
 	</joint>
   </xacro:macro>
@@ -40,5 +40,5 @@
     </link>
     <joint name="${name}_foot_joint" type="fixed">
-      <insert_block name="origin" />
+      <xacro:insert_block name="origin" />
       <parent link="${parent}"/>
       <child link="${name}_foot_link"/>

File: youbot_common/youbot_description/urdf/sensors/hokuyo_urg04_laser.urdf.xacro (robot description, xacro)
@@ -4,9 +4,9 @@
        xmlns:interface="http://playerstage.sourceforge.net/gazebo/xmlschema/#interface"
        xmlns:xacro="http://ros.org/wiki/xacro">
-  <include filename="$(find youbot_description)/urdf/sensors/hokuyo_urg04_laser.gazebo.xacro" />
+  <xacro:include filename="$(find youbot_description)/urdf/sensors/hokuyo_urg04_laser.gazebo.xacro" />
   <xacro:macro name="hokuyo_urg04_laser" params="name parent *origin ros_topic update_rate min_angle max_angle">
     <joint name="${name}_hokuyo_urg04_laser_joint" type="fixed">
       <axis xyz="0 1 0" />
-      <insert_block name="origin" />
+      <xacro:insert_block name="origin" />
       <parent link="${parent}_link"/>
       <child link="${name}_link"/>

File: youbot_common/youbot_description/urdf/sensors/kinect_camera.urdf.xacro (robot description, xacro)
@@ -4,8 +4,8 @@
       xmlns:interface="http://playerstage.sourceforge.net/gazebo/xmlschema/#interface"
       xmlns:xacro="http://ros.org/wiki/xacro">
-  <include filename="$(find youbot_description)/urdf/sensors/kinect_camera.gazebo.xacro"/>
+  <xacro:include filename="$(find youbot_description)/urdf/sensors/kinect_camera.gazebo.xacro"/>
   <xacro:macro name="kinect_camera" params="name parent *origin">
    <joint name="${name}_camera_joint" type="fixed">
-    <insert_block name="origin" />
+    <xacro:insert_block name="origin" />
     <parent link="${parent}" />
     <child link="${name}_camera" />

File: youbot_common/youbot_description/urdf/sensors/microsoft_lifecam.urdf.xacro (robot description, xacro)
@@ -4,8 +4,8 @@
       xmlns:interface="http://playerstage.sourceforge.net/gazebo/xmlschema/#interface"
       xmlns:xacro="http://ros.org/wiki/xacro">
-  <include filename="$(find youbot_description)/urdf/sensors/microsoft_lifecam.gazebo.xacro"/>
+  <xacro:include filename="$(find youbot_description)/urdf/sensors/microsoft_lifecam.gazebo.xacro"/>
   <xacro:macro name="microsoft_lifecam" params="name parent *origin">
    <joint name="${name}_camera_joint" type="fixed">
-    <insert_block name="origin" />
+    <xacro:insert_block name="origin" />
     <parent link="${parent}" />
     <child link="${name}_camera" />

File: youbot_common/youbot_description/urdf/youbot_arm/arm.urdf.xacro (robot description, xacro)
@@ -4,11 +4,11 @@
         xmlns:interface="http://playerstage.sourceforge.net/gazebo/xmlschema/#interface"
         xmlns:xacro="http://ros.org/wiki/xacro">
-	<include filename="$(find youbot_description)/urdf/youbot_arm/arm.gazebo.xacro" />
-	<include filename="$(find youbot_description)/urdf/youbot_arm/arm.transmission.xacro" />
-        <include filename="$(find youbot_description)/urdf/youbot_arm/limits.urdf.xacro" />
+	<xacro:include filename="$(find youbot_description)/urdf/youbot_arm/arm.gazebo.xacro" />
+	<xacro:include filename="$(find youbot_description)/urdf/youbot_arm/arm.transmission.xacro" />
+        <xacro:include filename="$(find youbot_description)/urdf/youbot_arm/limits.urdf.xacro" />
 	<xacro:macro name="youbot_arm" params="parent name *origin">
 		<!-- joint between base_link and arm_0_link -->
 		<joint name="${name}_joint_0" type="fixed" >
-			<insert_block name="origin" />
+			<xacro:insert_block name="origin" />
 			<parent link="${parent}" />
 			<child link="${name}_link_0" />

File: youbot_common/youbot_description/urdf/youbot_base/base.transmission.xacro (robot description, xacro)
@@ -4,7 +4,7 @@
        xmlns:interface="http://playerstage.sourceforge.net/gazebo/xmlschema/#interface"
        xmlns:xacro="http://ros.org/wiki/xacro">
-	<property name="wheel_mechanical_reduction" value="${624/35 * 80/18}" />
-	<property name="caster_mechanical_reduction" value="${624/35 * 80/18}" />
-  	<property name="" value="0.360" />
+	<xacro:property name="wheel_mechanical_reduction" value="${624/35 * 80/18}" />
+	<xacro:property name="caster_mechanical_reduction" value="${624/35 * 80/18}" />
+  	<!--<xacro:property name="" value="0.360" />-->
 	<xacro:macro name="youbot_base_transmission">
 	<!-- front left wheel -->

File: youbot_common/youbot_description/urdf/youbot_base/base.urdf.xacro (robot description, xacro)
@@ -5,32 +5,32 @@
         xmlns:xacro="http://ros.org/wiki/xacro">
 	<!-- sensors -->
-	<include filename="$(find youbot_description)/urdf/sensors/hokuyo_urg04_laser.urdf.xacro"/>
-	<include filename="$(find youbot_description)/urdf/youbot_base/base.gazebo.xacro" />
-	<include filename="$(find youbot_description)/urdf/youbot_base/base.transmission.xacro" />
+	<xacro:include filename="$(find youbot_description)/urdf/sensors/hokuyo_urg04_laser.urdf.xacro"/>
+	<xacro:include filename="$(find youbot_description)/urdf/youbot_base/base.gazebo.xacro" />
+	<xacro:include filename="$(find youbot_description)/urdf/youbot_base/base.transmission.xacro" />
  	<!-- simplified box collision geometry for base -->
-  	<property name="base_size_x" value="0.570" />
-  	<property name="base_size_y" value="0.360" />
-  	<property name="base_size_z" value="0.100" />
-	<property name="base_mass" value="22.0" />
-	<property name="caster_offset_x" value="0.228"  />
-  	<property name="caster_offset_y" value="0.158"  />
-  	<property name="caster_offset_z" value="-0.034" />
-	<property name="caster_mass" value="0.1" />
-	<property name="wheel_offset_x" value="0.0"  />
-  	<property name="wheel_offset_y" value="0.0"  />
-  	<property name="wheel_offset_z" value="0.0" />
-	<property name="wheel_mass" value="0.4" />
-	<property name="wheel_radius" value="0.05" />
-	<property name="wheel_length" value="0.005" />
-	<property name="caster_joint_damping" value="1.0" />
-	<property name="caster_joint_friction" value="1.0" />
-	<property name="caster_joint_effort" value="30" />
-	<property name="caster_joint_velocity" value="10" />
-	<property name="caster_joint_safety_k_velocity" value="10.0" />
-	<property name="wheel_joint_damping" value="1.0" />
-	<property name="wheel_joint_friction" value="1.0" />
-	<property name="wheel_joint_effort" value="30" />
-	<property name="wheel_joint_velocity" value="10" />
-	<property name="wheel_joint_safety_k_velocity" value="10.0" />
+  	<xacro:property name="base_size_x" value="0.570" />
+  	<xacro:property name="base_size_y" value="0.360" />
+  	<xacro:property name="base_size_z" value="0.100" />
+	<xacro:property name="base_mass" value="22.0" />
+	<xacro:property name="caster_offset_x" value="0.228"  />
+  	<xacro:property name="caster_offset_y" value="0.158"  />
+  	<xacro:property name="caster_offset_z" value="-0.034" />
+	<xacro:property name="caster_mass" value="0.1" />
+	<xacro:property name="wheel_offset_x" value="0.0"  />
+  	<xacro:property name="wheel_offset_y" value="0.0"  />
+  	<xacro:property name="wheel_offset_z" value="0.0" />
+	<xacro:property name="wheel_mass" value="0.4" />
+	<xacro:property name="wheel_radius" value="0.05" />
+	<xacro:property name="wheel_length" value="0.005" />
+	<xacro:property name="caster_joint_damping" value="1.0" />
+	<xacro:property name="caster_joint_friction" value="1.0" />
+	<xacro:property name="caster_joint_effort" value="30" />
+	<xacro:property name="caster_joint_velocity" value="10" />
+	<xacro:property name="caster_joint_safety_k_velocity" value="10.0" />
+	<xacro:property name="wheel_joint_damping" value="1.0" />
+	<xacro:property name="wheel_joint_friction" value="1.0" />
+	<xacro:property name="wheel_joint_effort" value="30" />
+	<xacro:property name="wheel_joint_velocity" value="10" />
+	<xacro:property name="wheel_joint_safety_k_velocity" value="10.0" />
 	<xacro:macro name="youbot_base" params="name">
 		<link name="${name}_footprint">

File: youbot_common/youbot_description/urdf/youbot_gripper/gripper.urdf.xacro (robot description, xacro)
@@ -4,11 +4,11 @@
        xmlns:interface="http://playerstage.sourceforge.net/gazebo/xmlschema/#interface"
        xmlns:xacro="http://ros.org/wiki/xacro">
-	<include filename="$(find youbot_description)/urdf/youbot_gripper/gripper.gazebo.xacro" />
-	<include filename="$(find youbot_description)/urdf/youbot_gripper/gripper.transmission.xacro" />
-	<include filename="$(find youbot_description)/urdf/youbot_gripper/limits.urdf.xacro" />
+	<xacro:include filename="$(find youbot_description)/urdf/youbot_gripper/gripper.gazebo.xacro" />
+	<xacro:include filename="$(find youbot_description)/urdf/youbot_gripper/gripper.transmission.xacro" />
+	<xacro:include filename="$(find youbot_description)/urdf/youbot_gripper/limits.urdf.xacro" />
 	<xacro:macro name="youbot_gripper" params="parent name *origin">
 		<!-- joint between arm_7_link and sdh_palm_link -->
 		<joint name="${name}_palm_joint" type="fixed" >
-			<insert_block name="origin" />
+			<xacro:insert_block name="origin" />
 			<parent link="${parent}" />
 			<child link="${name}_palm_link" />
