Commit message: added camera for rviz

File: youbot_common/youbot_description/urdf/youbot_arm/arm.urdf.xacro (robot description, xacro)
@@ -7,4 +7,5 @@
 	<xacro:include filename="$(find youbot_description)/urdf/youbot_arm/arm.transmission.xacro" />
         <xacro:include filename="$(find youbot_description)/urdf/youbot_arm/limits.urdf.xacro" />
+	<xacro:include filename="$(find youbot_description)/urdf/sensors/yb_cam.urdf.xacro" />
 	<xacro:macro name="youbot_arm" params="parent name *origin">
 		<!-- joint between base_link and arm_0_link -->
@@ -211,4 +212,7 @@
 			</collision>
 		</link>
+		<xacro:yb_cam name="${name}_cam" parent="${name}_link_5" >
+     			 <origin xyz="0.01 0 0.00" rpy="0 0 0" />
+    		</xacro:yb_cam>
 		<!-- extensions -->
 		<xacro:youbot_arm_gazebo name="${name}" />
