Commit message: visual changes

File: youbot_common/youbot_description/urdf/sensors/yb_cam.urdf.xacro (robot description, xacro)
@@ -19,5 +19,5 @@
     </inertial>
     <visual>
-      <origin xyz="0.0 0.0 0.0" rpy="0.0 0.0 ${M_PI/2}" />
+      <origin xyz="-0.036 +0.025 0.01" rpy="${M_PI/2} ${M_PI} ${M_PI/2}" />
       <geometry>
        <mesh filename="package://youbot_description/meshes/sensors/yb_cam.stl" scale="0.001 0.001 0.001"/>

File: youbot_common/youbot_description/urdf/youbot_arm/arm.urdf.xacro (robot description, xacro)
@@ -213,5 +213,5 @@
 		</link>
 		<xacro:yb_cam name="${name}_cam" parent="${name}_link_5" >
-     			 <origin xyz="0.01 0 0.00" rpy="0 0 0" />
+     			 <origin xyz="0.1 0 0.00" rpy="0 0 0" />
     		</xacro:yb_cam>
 		<!-- extensions -->
